File: hardware/servo/servo.kicad_sch (KiCad schematic)
At the start: 5 parts, among them J2 Conn_ARM_SWD_TagConnect_TC203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, U3 DRV8876PWPR, U4 STM32G030F6P6, U5 SIT3088EEUA

Commit message: hardware
Parts:
- added C10, C13, C8, C9: 100nF, Capacitor_SMD:C_0402_1005Metric, symbol Device:C
- added C11: 22nF, Capacitor_SMD:C_0402_1005Metric, symbol Device:C
- added C12: 220uF/50V, Capacitor_SMD:CP_Elec_10x10.5, symbol Device:CP
- added J3: Motor, Connector_JST:JST_PH_B2B-PH-K_1x02_P2.00mm_Vertical, symbol Connector_Generic:Conn_01x02
- added R10, R11, R12, R13, R14, R7, R8, R9: 10k, Resistor_SMD:R_0402_1005Metric, symbol Device:R
Connections:
- net +3.3V: now also C7.1, C10.1, C8.1, C9.1, R11.1, R12.1, R7.1, R8.1, R9.1
- net GND: now also C7.2, U3.5 (VREF), C10.2, C12.2, C13.2, C8.2, C9.2, R10.2, R14.1
- net VPP: now also C12.1
- net nFAULT: now reaches U4.1 (PB7)
- net nFAULT: now also U3.4 (~{FAULT}), R7.2
- net at U4.12 (PA4): now also U3.2 (PH/IN2)
- net at U4.14 (PA6): now also U3.1 (EN/IN1)
- net at U4.17 (PA11): now also U5.4 (DI)
- net at U4.18 (PA12): now also U5.1 (RO)
- net SCL: now reaches U4.2 (PB8)
- net SCL: now also R12.2
- net SDA: now reaches U4.3 (PB9)
- net SDA: now also R11.2
- net DE: now reaches U4.7 (PA1)
- net DE: now also U5.3 (DE), R13.2
- net at U5.2 (~{RE}): now also R13.1, R14.2
- net at U3.10 (OUT2): now also J3.2 (Pin_2)
- net at U3.12 (VCP): now also C13.1
- net at U3.13 (CPH): now also C11.1
- net at U3.14 (CPL): now also C11.2
- net at U3.16 (PMODE): now also R9.2
- net at U3.3 (~{SLEEP}): now also R8.2
- net at U3.7 (IMODE): now also R10.1
- net at U3.8 (OUT1): now also J3.1 (Pin_1)
Other:
- moved on the sheet: J2, U4, U5

Commit message: hardware
Parts:
- added D1: LED_R, LED_SMD:LED_0603_1608Metric, symbol Device:LED
- added JI2C1: Conn_01x04, Connector_JST:JST_PH_B4B-PH-K_1x04_P2.00mm_Vertical, symbol Connector_Generic:Conn_01x04
- added JLIM2: Limit, Connector_JST:JST_PH_B2B-PH-K_1x02_P2.00mm_Vertical, symbol Connector_Generic:Conn_01x02
- added JSERVO0, JSERVO1, JSERVO2, JSERVO3: Conn_01x03, Connector_JST:JST_PH_B3B-PH-K_1x03_P2.00mm_Vertical, symbol Connector_Generic:Conn_01x03
- added R15: 1k, Resistor_SMD:R_0402_1005Metric, symbol Device:R
- added R16, R17, R18, R19: 100R, Resistor_SMD:R_0402_1005Metric, symbol Device:R
- added R20: 10k, Resistor_SMD:R_0402_1005Metric, symbol Device:R
- added U6: SRV05-4, Package_TO_SOT_SMD:SOT-23-6, symbol Power_Protection:SRV05-4
- renumbered J3 to JMOTOR2
Connections:
- net +3.3V: now also D1.2 (A), JI2C1.1 (Pin_1), R20.1, U6.5 (VCC)
- net GND: now also JI2C1.4 (Pin_4), JLIM2.2 (Pin_2), JSERVO0.3 (Pin_3), JSERVO1.3 (Pin_3), JSERVO2.3 (Pin_3), JSERVO3.3 (Pin_3), U6.2 (GND)
- net SCL: now also JI2C1.3 (Pin_3)
- net SDA: now also JI2C1.2 (Pin_2)
- net VPP: now also JSERVO0.1 (Pin_1), JSERVO1.1 (Pin_1), JSERVO2.1 (Pin_1), JSERVO3.1 (Pin_1)
- net SERVO2: now reaches U4.11 (PA3)
- net SERVO2: now also R17.1, U6.4 (IO3)
- net LED: now reaches U4.13 (PA5)
- net LED: now also R15.1
- net SERVO3: now reaches U4.15 (PA7)
- net SERVO3: now also R16.1, U6.6 (IO4)
- net at U4.16 (PA8): now also JLIM2.1 (Pin_1), R20.2
- net SERVO0: now reaches U4.6 (PA0)
- net SERVO0: now also R18.2, U6.1 (IO1)
- net SERVO1: now reaches U4.8 (PA2)
- net SERVO1: now also R19.2, U6.3 (IO2)
- new net: JSERVO3.2 (Pin_2), R16.2
- new net: JSERVO1.2 (Pin_2), R19.1
- new net: JSERVO0.2 (Pin_2), R18.1
- new net: D1.1 (K), R15.2
- new net: JSERVO2.2 (Pin_2), R17.2
Other:
- moved on the sheet: C8, C9

Commit message: hardware
Parts:
- added D2: SS36, Diode_SMD:D_SMA, symbol Device:D_Schottky
- added H2, H3, H4, H5: MountingHole, MountingHole:MountingHole_3.2mm_M3_Pad_TopBottom, symbol Mechanical:MountingHole
- added JBUS1, JBUS2: Conn_01x04_XH, Connector_JST:JST_XH_S4B-XH-A_1x04_P2.50mm_Horizontal, symbol Connector_Generic:Conn_01x04
- added JPWR2: Conn_01x02_XH, Connector_JST:JST_XH_S2B-XH-A_1x02_P2.50mm_Horizontal, symbol Connector_Generic:Conn_01x02
Connections:
- net GND: now also JBUS1.4 (Pin_4), JBUS2.4 (Pin_4), JPWR2.2 (Pin_2)
- net VPP: now also D2.1 (K), JBUS1.1 (Pin_1), JBUS2.1 (Pin_1)
- net at U5.6 (A): now also JBUS1.3 (Pin_3), JBUS2.3 (Pin_3)
- net at U5.7 (B): now also JBUS1.2 (Pin_2), JBUS2.2 (Pin_2)
- new net: D2.2 (A), JPWR2.1 (Pin_1)
Other:
- moved on the sheet: C7

Commit message: updates
Parts:
- added JPTERM: TERM, Jumper:SolderJumper-2_P1.3mm_Open_Pad1.0x1.5mm, symbol Jumper:SolderJumper_2_Open
- added R21: 120R, Resistor_SMD:R_1206_3216Metric, symbol Device:R
Connections:
- net B: now reaches JBUS1.2 (Pin_2), JBUS2.2 (Pin_2), U5.7 (B)
- net B: now also R21.2
- net A: now reaches JBUS1.3 (Pin_3), JBUS2.3 (Pin_3), U5.6 (A)
- net A: now also JPTERM.2 (B)
- new net: JPTERM.1 (A), R21.1

Commit message: updates
Parts:
- renumbered JPTERM to JPTERM2
Changed lines of the file:
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@@
 		(in_pos_files yes)
 		(dnp no)
-		(property "Reference" "JPTERM"
+		(property "Reference" "JPTERM2"
 			(at 354.076 217.17 90)
 			(show_name no)
@@
 			(project "servo"
 				(path "/e63e39d7-6ac0-4ffd-8aa3-1841a4541b55"
-					(reference "JPTERM")
+					(reference "JPTERM2")
 					(unit 1)
 				)

Commit message: boms
Parts:
- added D3: SS36, Diode_SMD:D_SMA, symbol Device:D_Schottky
- added JP2, JP3, JP4: SolderJumper_3_Bridged12, Jumper:SolderJumper-3_P1.3mm_Bridged12_RoundedPad1.0x1.5mm, symbol Jumper:SolderJumper_3_Bridged12
- JPTERM2: footprint Jumper:SolderJumper-2_P1.3mm_Open_Pad1.0x1.5mm -> (none); now left out of the parts list
Connections:
- net VPP: now also D3.1 (K), JP2.3 (B), JP3.3 (B), JP4.1 (A); no longer JBUS1.1 (Pin_1), JBUS2.1 (Pin_1), JSERVO0.1 (Pin_1), JSERVO1.1 (Pin_1), JSERVO2.1 (Pin_1), JSERVO3.1 (Pin_1), U3.11 (VM)
- new net: D3.2 (A), JBUS1.1 (Pin_1), JBUS2.1 (Pin_1)
- new net: JP4.2 (C), U3.11 (VM)
- new net +5V: JP2.1 (A), JP3.1 (A), JP4.3 (B)
- new net SP1: JP2.2 (C), JSERVO0.1 (Pin_1), JSERVO1.1 (Pin_1)
- new net SP2: JP3.2 (C), JSERVO2.1 (Pin_1), JSERVO3.1 (Pin_1)
Other:
- added sheet PSU_SERVO (psu_servo.kicad_sch)
- moved on the sheet: D1, JSERVO0, JSERVO1, JSERVO2, JSERVO3, R15, R16, R17, R18, R19, U6

Commit message: ministepper: finalize pin map + sync firmware to hardware rev 0.1
Hardware (schematic + docs) and firmware now share a single source of
truth for the STM32G071G8U6 UFQFPN-28 pinout:

- USART2 on PA2/PA3 (RS-485) — dedicated pins, no SYSCFG remap needed
  (unlike the servo's STM32G030 where PA11/PA12 shared pads with
  PA9/PA10)
- Two independent step timers: TIM1_CH1 on PA8 (STEP1) and TIM2_CH1
  on PA0 (STEP2) — each axis can run at its own rate
- Shared SPI1 (PA5/6/7) to both TMC2130s with software-managed CS on
  PA4 (TMC1) and PA12 (TMC2)
- Shared DRV_ENN on PA11 — pulls both drivers in/out of enable at once
- Per-axis limit switches (PB0, PB3) and DIAG1 stall/fault inputs
  (PB1, PB4)
- I2C1 on PB6/PB7 for expansion
- Status LED on PB5 (moved off PA5 which is now SPI SCK)
- 1 spare GPIO (PB8) for future use

firmware/tsumikoro-ministepper/src/main.c rewritten:
- Switched from USART1 to USART2; DMA request IDs updated
- PIN_* defines added for every pin from the schematic, cross-referenced
  to the hardware doc
- GPIO init configures all driver control lines (CS high, DRV_ENN high
  = off at boot), DIAG inputs, limit inputs with pull-ups, and the DE
  line for RS-485 (starts low = RX)
- Error_Handler moved to LED on PB5
- Bus callback extended to two-axis selector (byte 0 of move/stop
  payload picks axis 1 or 2); GET_STATUS reports both positions
- SPI1 / TIM1 / TIM2 stepper peripheral init still TODO — the real
  step generator will come with the SPI driver + per-axis motion
  planner

Hardware docs:
- CLAUDE.md adds "Ministepper PCB Pin Map" section (authoritative)
- hardware/ministepper/docs/README.md pin map updated to the final
  layout with independent STEP timers; sense-resistor variants
  (0.1 ohm standard vs 0.68 ohm micro / 28BYJ-48) documented
- hardware/TODO.md marks pin map + firmware sync done

Firmware builds clean (23 KB flash, 14.7 KB RAM) on STM32G071G8U6.
Parts:
- added R25: 10k, Resistor_SMD:R_0402_1005Metric, symbol Device:R
Connections:
- net +3.3V: now also R25.1
- net at J2.3 (~{RESET}), U4.4 (NRST): now also R25.2
Changed lines of the file:
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@@
 	)
 	(junction
+		(at 196.85 146.05)
+		(diameter 0)
+		(color 0 0 0 0)
+	)
+	(junction
 		(at 288.29 205.74)
 		(diameter 0)
@@
 	(wire
 		(pts
+			(xy 189.23 146.05) (xy 196.85 146.05)
+		)
+		(stroke
+			(width 0)
+			(type default)
+		)
+	)
+	(wire
+		(pts
 			(xy 246.38 190.5) (xy 247.65 190.5)
 		)
@@
 	(wire
 		(pts
+			(xy 189.23 143.51) (xy 189.23 146.05)
+		)
+		(stroke
+			(width 0)
+			(type default)
+		)
+	)
+	(wire
+		(pts
 			(xy 246.38 110.49) (xy 250.19 110.49)
 		)
@@
 	(wire
 		(pts
+			(xy 189.23 134.62) (xy 189.23 135.89)
+		)
+		(stroke
+			(width 0)
+			(type default)
+		)
+	)
+	(wire
+		(pts
 			(xy 306.07 153.67) (xy 306.07 165.1)
 		)
@@
 	(wire
 		(pts
-			(xy 196.85 154.94) (xy 196.85 135.89)
+			(xy 196.85 154.94) (xy 196.85 146.05)
 		)
 		(stroke
@@
 	(wire
 		(pts
+			(xy 196.85 146.05) (xy 196.85 135.89)
+		)
+		(stroke
+			(width 0)
+			(type default)
+		)
+	)
+	(wire
+		(pts
 			(xy 200.66 222.25) (xy 209.55 222.25)
 		)
@@
 	)
 	(symbol
+		(lib_id "Device:R")
+		(at 189.23 139.7 0)
+		(unit 1)
+		(body_style 1)
+		(exclude_from_sim no)
+		(in_bom yes)
+		(on_board yes)
+		(in_pos_files yes)
+		(dnp no)
+		(property "Reference" "R25"
+			(at 191.77 137.16 0)
+			(show_name no)
+			(do_not_autoplace no)
+			(effects
+				(font
+					(size 1.27 1.27)
+				)
+				(justify left)
+			)
+		)
+		(property "Value" "10k"
+			(at 191.77 142.24 0)
+			(show_name no)
+			(do_not_autoplace no)
+			(effects
+				(font
+					(size 1.27 1.27)
+				)
+				(justify left)
+			)
+		)
+		(property "Footprint" "Resistor_SMD:R_0402_1005Metric"
+			(at 189.23 139.7 0)
+			(hide yes)
+			(show_name no)
+			(do_not_autoplace no)
+			(effects
+				(font
+					(size 1.27 1.27)
+				)
+			)
+		)
+		(property "Datasheet" ""
+			(at 189.23 139.7 0)
+			(hide yes)
+			(show_name no)
+			(do_not_autoplace no)
+			(effects
+				(font
+					(size 1.27 1.27)
+				)
+			)
+		)
+		(property "Description" "Feedback divider bottom resistor (BASIC)"
+			(at 189.23 139.7 0)
+			(hide yes)
+			(show_name no)
+			(do_not_autoplace no)
+			(effects
+				(font
+					(size 1.27 1.27)
+				)
+			)
+		)
+		(property "LCSC" "C25744"
+			(at 189.23 139.7 0)
+			(hide yes)
+			(show_name no)
+			(do_not_autoplace no)
+			(effects
+				(font
+					(size 1.27 1.27)
+				)
+			)
+		)
+		(property "MPN" "0402WGF1002TCE"
+			(at 189.23 139.7 0)
+			(hide yes)
+			(show_name no)
+			(do_not_autoplace no)
+			(effects
+				(font
+					(size 1.27 1.27)
+				)
+			)
+		)
+		(property "Manufacturer" "UNI-ROYAL"
+			(at 189.23 139.7 0)
+			(hide yes)
+			(show_name no)
+			(do_not_autoplace no)
+			(effects
+				(font
+					(size 1.27 1.27)
+				)
+			)
+		)
+		(pin "1"
+		)
+		(pin "2"
+		)
+		(instances
+			(project "servo"
+				(path "/e63e39d7-6ac0-4ffd-8aa3-1841a4541b55"
+					(reference "R25")
+					(unit 1)
+				)
+			)
+		)
+	)
+	(symbol
 		(lib_id "power:+3.3V")
 		(at 223.52 115.57 0)
@@
 					(unit 1)
 				)
+			)
+		)
+	)
+	(symbol
+		(lib_id "power:+3.3V")
+		(at 189.23 134.62 0)
+		(unit 1)
+		(body_style 1)
+		(exclude_from_sim no)
+		(in_bom yes)
+		(on_board yes)
+		(in_pos_files yes)
+		(dnp no)
+		(fields_autoplaced yes)
+		(property "Reference" "#PWR053"
+			(at 189.23 138.43 0)
+			(hide yes)
+			(show_name no)
+			(do_not_autoplace no)
+			(effects
+				(font
+					(size 1.27 1.27)
+				)
+			)
+		)
+		(property "Value" "+3.3V"
+			(at 189.23 129.54 0)
+			(show_name no)
+			(do_not_autoplace no)
+			(effects
+				(font
+					(size 1.27 1.27)
+				)
+			)
+		)
+		(property "Footprint" ""
+			(at 189.23 134.62 0)
+			(hide yes)
+			(show_name no)
+			(do_not_autoplace no)
+			(effects
+				(font
+					(size 1.27 1.27)
+				)
+			)
+		)
+		(property "Datasheet" ""
+			(at 189.23 134.62 0)
+			(hide yes)
+			(show_name no)
+			(do_not_autoplace no)
+			(effects
+				(font
+					(size 1.27 1.27)
+				)
+			)
+		)
+		(property "Description" "Power symbol creates a global label with name \"+3.3V\""
+			(at 189.23 134.62 0)
+			(hide yes)
+			(show_name no)
+			(do_not_autoplace no)
+			(effects
+				(font
+					(size 1.27 1.27)
+				)
+			)
+		)
+		(pin "1"
+		)
+		(instances
+			(project "servo"
+				(path "/e63e39d7-6ac0-4ffd-8aa3-1841a4541b55"
+					(reference "#PWR053")
+					(unit 1)
+				)
