File: hardware/servo/servo.kicad_sch (KiCad schematic)
At the start: 49 parts, among them J2 Conn_ARM_SWD_TagConnect_TC203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, U3 DRV8876PWPR, U4 STM32G030F6P6, U5 SIT3088EEUA, U6 SRV05-4

Commit message: hw: swap 100nF 16V (C1525) → 100nF 50V (C307331) across all boards
Standardizes on 50V-rated 100nF 0402 for all bypass/decoupling caps.
Required on ministepper for VS/VSA/VCP nets (up to ~51V on charge
pump); applied across servo and bridge too for BOM consistency. Both
are JLCPCB basic parts — no assembly fee change.

Regenerated docs + JLCPCB packages.

Co-Authored-By: Claude Opus 4.6 (1M context) <noreply@anthropic.com>
Parts:
- C10, C13, C7, C8, C9: LCSC C1525 -> C307331; MPN CL05B104KO5NNNC -> CL05B104KB54PNC
Changed lines of the file:
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@@
 			)
 		)
-		(property "LCSC" "C1525"
+		(property "LCSC" "C307331"
 			(at 185.42 110.49 0)
 			(hide yes)
@@
 			)
 		)
-		(property "MPN" "CL05B104KO5NNNC"
+		(property "MPN" "CL05B104KB54PNC"
 			(at 185.42 110.49 0)
 			(hide yes)
@@
 			)
 		)
-		(property "LCSC" "C1525"
+		(property "LCSC" "C307331"
 			(at 367.03 157.48 0)
 			(hide yes)
@@
 			)
 		)
-		(property "MPN" "CL05B104KO5NNNC"
+		(property "MPN" "CL05B104KB54PNC"
 			(at 367.03 157.48 0)
 			(hide yes)
@@
 			)
 		)
-		(property "LCSC" "C1525"
+		(property "LCSC" "C307331"
 			(at 175.26 110.49 0)
 			(hide yes)
@@
 			)
 		)
-		(property "MPN" "CL05B104KO5NNNC"
+		(property "MPN" "CL05B104KB54PNC"
 			(at 175.26 110.49 0)
 			(hide yes)
@@
 			)
 		)
-		(property "LCSC" "C1525"
+		(property "LCSC" "C307331"
 			(at 337.82 191.77 0)
 			(hide yes)
@@
 			)
 		)
-		(property "MPN" "CL05B104KO5NNNC"
+		(property "MPN" "CL05B104KB54PNC"
 			(at 337.82 191.77 0)
 			(hide yes)
@@
 			)
 		)
-		(property "LCSC" "C1525"
+		(property "LCSC" "C307331"
 			(at 170.18 140.97 0)
 			(hide yes)
@@
 			)
 		)
-		(property "MPN" "CL05B104KO5NNNC"
+		(property "MPN" "CL05B104KB54PNC"
 			(at 170.18 140.97 0)
 			(hide yes)
