File: hardware/servo/psu_servo.kicad_sch (KiCad schematic)
At the start: 10 parts, among them U7 LMR38020SDDAR

Commit message: hw: swap 100nF 16V (C1525) → 100nF 50V (C307331) across all boards
Standardizes on 50V-rated 100nF 0402 for all bypass/decoupling caps.
Required on ministepper for VS/VSA/VCP nets (up to ~51V on charge
pump); applied across servo and bridge too for BOM consistency. Both
are JLCPCB basic parts — no assembly fee change.

Regenerated docs + JLCPCB packages.

Co-Authored-By: Claude Opus 4.6 (1M context) <noreply@anthropic.com>
Parts:
- C27: LCSC C1525 -> C307331; MPN CL05B104KO5NNNC -> CL05B104KB54PNC
Changed lines of the file:
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@@
 			)
 		)
-		(property "Description" "Bootstrap cap BOOT-SW 100nF 16V X7R 0402 (BASIC)"
+		(property "Description" "Bootstrap cap BOOT-SW 100nF 50V X7R 0402 (BASIC)"
 			(at 160.02 66.04 0)
 			(hide yes)
@@
 			)
 		)
-		(property "LCSC" "C1525"
+		(property "LCSC" "C307331"
 			(at 160.02 66.04 0)
 			(hide yes)
@@
 			)
 		)
-		(property "MPN" "CL05B104KO5NNNC"
+		(property "MPN" "CL05B104KB54PNC"
 			(at 160.02 66.04 0)
 			(hide yes)
