File: hardware/servo/servo.kicad_pcb (KiCad board)
At the start: 4 copper layers, 62 x 45 mm, 72 parts, among them J2 Conn_ARM_SWD_TagConnect_TC203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, U2 TPS54061DRBT, U3 DRV8876PWPR, U4 STM32G030F6P6, U5 SIT3088EEUA, U6 SRV05-4, U7 LMR38020SDDAR

Commit message: hw+fw: fix STM32G071G8U6 UFQFPN28 symbol + pin map
The tsumikoro:STM32G071G8U6 symbol had a fabricated pin map that
didn't match ST DS12232 Figure 9 — VDD/VDDA were split onto pins 1/2
(they're actually fused on pin 3 on this package), NRST was assigned
to pin 3 (it's on pin 5), pin 28 was labelled VDD_2 (it's PB8), and
DIR2 was on PB2 (which is not bonded out on UFQFPN28).

Because the ministepper is not yet wired and firmware addresses GPIOs
by port name, no PCB damage resulted — but every pin number in docs,
firmware comments, and the symbol was off.

Rewritten against the datasheet:

- Symbol rebuilt with the real 29-pin UFQFPN28 layout (28 signal +
  EP), including PC14/PC15 on pins 1/2 and PC6 on pin 17.
- DIR2 reassigned from phantom PB2 to PC6 (pin 17).
- GPIOC clock enabled in firmware for PC6.
- CLAUDE.md and ministepper/docs/README.md pin tables rewritten.
- docs/README now calls out required MCU decoupling (100 nF + 4.7 µF
  bulk + NRST filter) that was implicitly missing when docs assumed
  two separate VDD pins.

Co-Authored-By: Claude Opus 4.6 (1M context) <noreply@anthropic.com>
Parts:
- added JPBOOT2: BOOT, Jumper:SolderJumper-2_P1.3mm_Open_Pad1.0x1.5mm, F.Cu at (93.2, 123.8)
- added R_BOOT0: 10k, Resistor_SMD:R_0402_1005Metric, F.Cu at (87.6, 115.3)
Routing:
- net Net-(J2-SWCLK): track 4.04 -> 24.1 mm, vias 0 -> 4
- net +3.3V: track 35.8 -> 37.3 mm, vias 14 -> 15
- net GND: track 21.6 -> 22.6 mm, vias 64 -> 65
