File: hardware/servo/servo.kicad_pcb (KiCad board)
At the start: 4 copper layers, 62 x 45 mm, 74 parts, among them J2 Conn_ARM_SWD_TagConnect_TC203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, U2 TPS54061DRBT, U3 DRV8876PWPR, U4 STM32G030F6P6, U5 SIT3088EEUA, U6 SRV05-4, U7 LMR38020SDDAR

Commit message: hw/servo: regen docs + JLCPCB package after rewire
Parts:
- removed R7: 10k, Resistor_SMD:R_0402_1005Metric
- moved C9 5.20 mm to (75.6, 115.8)
- moved R_BOOT0 0.30 mm to (87.6, 115.6)
Connections:
- J2 pad 2: Net-(J2-SWDIO) -> /SWDIO
- J2 pad 4: Net-(J2-SWCLK) -> /SWCLK
- JPBOOT2 pad 1: Net-(J2-SWCLK) -> /SWCLK
- R_BOOT0 pad 1: Net-(J2-SWCLK) -> /SWCLK
- U3 pad 1: Net-(U3-EN/IN1) -> /EN
- U3 pad 2: Net-(U3-PH/IN2) -> /PH
- U3 pad 4: /nFAULT -> unconnected-(U3-~{FAULT}-Pad4)
- U4 pad 1: /nFAULT -> /SCL
- U4 pad 10: +3.3V -> /SERVO2
- U4 pad 11: /SERVO2 -> /PH
- U4 pad 12: Net-(U3-PH/IN2) -> /LED
- U4 pad 13: /LED -> /EN
- U4 pad 14: Net-(U3-EN/IN1) -> /SERVO3
- U4 pad 15: /SERVO3 -> Net-(JLIM2-Pin_1)
- U4 pad 16: Net-(JLIM2-Pin_1) -> Net-(U4-PA11[PA9])
- U4 pad 17: Net-(U4-PA11) -> Net-(U4-PA12[PA10])
- U4 pad 18: Net-(U4-PA12) -> /SWDIO
- U4 pad 19: Net-(J2-SWDIO) -> /SWCLK
- U4 pad 2: /SCL -> /SDA
- U4 pad 20: Net-(J2-SWCLK) -> unconnected-(U4-PB3/PB4/PB5/PB6-Pad20)
- U4 pad 3: /SDA -> unconnected-(U4-PC15/OSC32_OUT-Pad3)
- U4 pad 4: Net-(J2-~{RESET}) -> +3.3V
- U4 pad 5: +3.3V -> GND
- U4 pad 6: /SERVO0 -> Net-(J2-~{RESET})
- U4 pad 7: /DE -> /SERVO0
- U4 pad 8: /SERVO1 -> /DE
- U4 pad 9: GND -> /SERVO1
- U5 pad 1: Net-(U4-PA12) -> Net-(U4-PA12[PA10])
- U5 pad 4: Net-(U4-PA11) -> Net-(U4-PA11[PA9])
Routing:
- net /SWCLK: track 0.00 -> 24.7 mm, vias 0 -> 4
- net Net-(J2-SWCLK): track 24.1 -> 0.00 mm, vias 4 -> 0
- net Net-(U3-EN/IN1): track 12.0 -> 0.00 mm, vias 2 -> 0
- net /EN: track 0.00 -> 11.7 mm, vias 0 -> 2
- net Net-(U3-PH/IN2): track 11.6 -> 0.00 mm, vias 2 -> 0
- net /PH: track 0.00 -> 11.6 mm, vias 0 -> 2
- net Net-(U4-PA11): track 7.22 -> 0.00 mm
- net Net-(U4-PA11[PA9]): track 0.00 -> 6.61 mm
- net /nFAULT: track 6.47 -> 0.00 mm
- net /SWDIO: track 0.00 -> 5.85 mm
- net Net-(J2-SWDIO): track 5.58 -> 0.00 mm
- net Net-(U4-PA12[PA10]): track 0.00 -> 5.45 mm
- net Net-(U4-PA12): track 4.98 -> 0.00 mm
- net /SERVO1: track 34.7 -> 31.6 mm
- net +3.3V: track 37.3 -> 35.6 mm, vias 15 -> 13
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