File: hardware/bridge/bridge.kicad_pcb (KiCad board)
At the start: 4 copper layers, 0 parts

Commit message: hardware: scaffold ministepper (TMC2130 dual stepper driver) project
Third PCB in the family, matching firmware/tsumikoro-ministepper's
STM32G071G8U6 target. 4-layer, same JLC04161H stackup and design rules
as servo + bridge.

Placed (not wired):
- U1 STM32G071G8U6 UFQFPN-28 (core MCU)
- U2, U3 TMC2130-LA-T (shared SPI bus, per-driver CS/STEP/DIR/EN/DIAG)
- U4 SIT3088EEUA (RS-485, USART2 on PA2/PA3 — no SYSCFG remap needed on
  G071 unlike G030)
- JBUS1, JBUS2 (JST-XH 4-pin daisy-chain, V+/B/A/GND)
- JMOT1, JMOT2 (JST-XH 4-pin stepper outputs)
- JPWR (JST-XH 2-pin optional external motor supply)
- D1, D2 (SS34 Schottky diode-OR for bus V+ vs external)

PSU sub-sheet forked from servo's psu.kicad_sch — TPS54061 @ 3.3V,
sized for ~150 mA (MCU + 2x TMC VCC_IO + RS-485). UUIDs retargeted for
the ministepper project.

Docs README covers the full pin map, TMC2130 strapping checklist
(sense resistors, charge pump cap, VCP/5VOUT/VCC caps, DIAG pull-ups),
connectors, and regeneration commands.

Added hardware/TODO.md tracking servo/bridge/ministepper/light-sensor
projects with outstanding work per board.

Makefile PROJECTS list extended to servo bridge ministepper.
Parts:
- added C1: 2.2uF, Capacitor_SMD:C_1206_3216Metric, F.Cu at (170.7, 75.6)
- added C2: 100nF, Capacitor_SMD:C_0603_1608Metric, F.Cu at (169.9, 78.5)
- added C3: 100nF, Capacitor_SMD:C_0402_1005Metric, F.Cu at (160.9, 87.0)
- added C4: 10uF, Capacitor_SMD:C_0805_2012Metric, F.Cu at (167.3, 82.0)
- added C5: 10uF, Capacitor_SMD:C_0805_2012Metric, F.Cu at (167.3, 85.0)
- added D1: MBRD10200, Package_TO_SOT_SMD:TO-252-2, F.Cu at (152.2, 94.8)
- added D2: MBRD10200, Package_TO_SOT_SMD:TO-252-2, F.Cu at (152.2, 103.0)
- added JBUS1: Conn_01x04_XH, Connector_JST:JST_XH_S4B-XH-A_1x04_P2.50mm_Horizontal, F.Cu at (134.3, 94.0)
- added JBUS2: Conn_01x04_XH, Connector_JST:JST_XH_S4B-XH-A_1x04_P2.50mm_Horizontal, F.Cu at (134.3, 107.5)
- added JDC1: DC-005 2.0mm, Connector_BarrelJack:BarrelJack_GCT_DCJ200-10-A_Horizontal, F.Cu at (119.2, 75.9)
- added JDC2: DC-005 2.0mm, Connector_BarrelJack:BarrelJack_GCT_DCJ200-10-A_Horizontal, F.Cu at (131.6, 75.9)
- added JPTERM1: TERM1, Jumper:SolderJumper-2_P1.3mm_Open_Pad1.0x1.5mm, F.Cu at (154.7, 84.9)
- added JPTERM2: TERM2, Jumper:SolderJumper-2_P1.3mm_Open_Pad1.0x1.5mm, F.Cu at (154.7, 88.4)
- added J_USB2: USB-TYPE-C-019, Connector_USB:USB_C_Receptacle_GCT_USB4105-xx-A_16P_TopMnt_Horizontal, F.Cu at (151.1, 112.3)
- added L1: 10uH, Inductor_SMD:L_Changjiang_FNR4030S, F.Cu at (162.2, 83.3)
- added R1: 100k, Resistor_SMD:R_0402_1005Metric, F.Cu at (171.0, 81.5)
- added R2: 22k, Resistor_SMD:R_0402_1005Metric, F.Cu at (171.0, 83.5)
- added R3: 10k, Resistor_SMD:R_0402_1005Metric, F.Cu at (171.0, 85.5)
- added R4: 120R, Resistor_SMD:R_1206_3216Metric, F.Cu at (149.8, 84.8)
- added R5: 120R, Resistor_SMD:R_1206_3216Metric, F.Cu at (149.8, 88.1)
- added R_BOOT2: 10k, Resistor_SMD:R_0402_1005Metric, F.Cu at (155.8, 74.9)
- added R_CC1: 5.1k, Resistor_SMD:R_0402_1005Metric, F.Cu at (155.8, 76.9)
- added R_CC2: 5.1k, Resistor_SMD:R_0402_1005Metric, F.Cu at (155.8, 78.9)
- added R_EN2: 10k, Resistor_SMD:R_0402_1005Metric, F.Cu at (155.8, 80.9)
- added SW_BOOT2: BOOT, tsumikoro:SW_Push_1P1T_XKB_TS-1187A, F.Cu at (142.7, 77.2)
- added SW_RESET2: RESET, tsumikoro:SW_Push_1P1T_XKB_TS-1187A, F.Cu at (142.7, 83.9)
- added U1: SIT3088EEUA, Package_SO:MSOP-8_3x3mm_P0.65mm, F.Cu at (150.7, 76.2)
- added U2: LMR38020SDDAR, Package_SO:SOIC-8-1EP_3.9x4.9mm_P1.27mm_EP2.29x3mm, F.Cu at (163.6, 77.3)
- added U3: SIT3088EEUA, Package_SO:MSOP-8_3x3mm_P0.65mm, F.Cu at (150.7, 80.8)
- added U4: ESP32-S3-MINI-1-N8, tsumikoro:ESP32-S3-MINI-1, F.Cu at (186.6, 117.8)
