File: hardware/ministepper/stepper_channel.kicad_sch (KiCad schematic)
At the start: 16 parts, among them U1 TMC2130-LA

Commit message: hw: swap 100nF 16V (C1525) → 100nF 50V (C307331) across all boards
Standardizes on 50V-rated 100nF 0402 for all bypass/decoupling caps.
Required on ministepper for VS/VSA/VCP nets (up to ~51V on charge
pump); applied across servo and bridge too for BOM consistency. Both
are JLCPCB basic parts — no assembly fee change.

Regenerated docs + JLCPCB packages.

Co-Authored-By: Claude Opus 4.6 (1M context) <noreply@anthropic.com>
Parts:
- C_AIN, C_BRA_FILT, C_BRB_FILT, C_VCC, C_VCP, C_VS, C_VSA: LCSC C1525 -> C307331; MPN CL05B104KO5NNNC -> CL05B104KB54PNC
Connections:
- net GND: now also C_BRA_FILT.2, C_BRB_FILT.2
- net at RSB.1, RSB_M.1, U1.14 (BRB): now also C_BRB_FILT.1
- net at U1.27 (CPO): now also C_CP.2
- net at U1.28 (CPI): now also C_CP.1
- net VCP: now reaches U1.29 (VCP)
- net at RSA.1, RSA_M.1, U1.33 (BRA): now also C_BRA_FILT.1
Other:
- moved on the sheet: C_CP, C_VCC, C_VCP

Commit message: hw/ministepper: align TMC2130 VCC/VCC_IO per datasheet
- Add R_VCC (2.2 ohm 0402, C321161) between 5VOUT and VCC per
  TMC2130 datasheet §3.2 — decouples charge-pump/digital noise from
  5VOUT, improving microstep/chopper performance.
- Change C_VCC: 100 nF 0402 → 470 nF 0603 25V X7R (C1623 basic) to
  match the datasheet's explicit spec on pin 26.
- Rename C_AIN → C_VCC_IO: datasheet recommends 100 nF on pin 8
  (VCC_IO). AIN_IREF is left open (self-biases to V5VOUT/2 per
  electrical characteristics; unused with external sense resistors +
  I_scale_analog=0).
- Regenerated docs + JLCPCB package.

Co-Authored-By: Claude Opus 4.6 (1M context) <noreply@anthropic.com>
Parts:
- added R_VCC: 2.2, Resistor_SMD:R_0402_1005Metric, symbol Device:R
- C_VCC: value 100nF -> 470nF; footprint Capacitor_SMD:C_0402_1005Metric -> Capacitor_SMD:C_0603_1608Metric; LCSC C307331 -> C1623; MPN CL05B104KB54PNC -> CL10B474KA8NNNC
- renumbered C_AIN to C_VCC_IO
Connections:
- net GND: now also C_VCC.1, C_VCC_IO.2, C_VS.2, C_VSA.2, C_VS_BULK.2
- net VCP: now also C_VCP.2
- net VPP: now reaches U1.16 (VS)
- net VPP: now also C_VCP.1, C_VS.1, C_VSA.1, C_VS_BULK.1, U1.30 (VSA), U1.31 (VS_2)
- net at C_5VOUT.1, U1.25 (5VOUT): now also R_VCC.1
- net 5VOUT: now reaches U1.26 (VCC)
- net 5VOUT: now also C_VCC.2, R_VCC.2
- net +3.3V: now reaches U1.8 (VCC_IO)
- net +3.3V: now also C_VCC_IO.1
Other:
- moved on the sheet: C_VCC, C_VCC_IO, C_VS, C_VSA, C_VS_BULK
