File: hardware/ministepper/stepper_channel.kicad_sch (KiCad schematic)
At the start: 17 parts, among them U1 TMC2130-LA

Commit message: pcb
Parts:
- renumbered C_5VOUT to C_5VOUT2, C_BRA_FILT to C_BRA_FILT2, C_BRB_FILT to C_BRB_FILT2, C_CP to C_CP2, C_VCC to C_VCC2, C_VCC_IO to C_VCC_IO2, C_VCP to C_VCP2, C_VS to C_VS2, C_VSA to C_VSA2, C_VS_BULK to C_VS_BULK2, RSA to RSA2, RSA_M to RSA_M2, RSB to RSB2, RSB_M to RSB_M2, R_VCC to R_VCC2, U1 to U2
Connections:
- net +3.3V: now also U2.10 (SPI_MODE)
- net +3V3: no longer U2.10 (SPI_MODE)

Commit message: Checkpoint
Parts:
- renumbered C_5VOUT2 to C_5VOUT3, C_BRA_FILT2 to C_BRA_FILT3, C_BRB_FILT2 to C_BRB_FILT3, C_CP2 to C_CP3, C_VCC2 to C_VCC3, C_VCC_IO2 to C_VCC_IO3, C_VCP2 to C_VCP3, C_VS2 to C_VS3, C_VSA2 to C_VSA3, C_VS_BULK2 to C_VS_BULK3, RSA2 to RSA3, RSA_M2 to RSA_M3, RSB2 to RSB3, RSB_M2 to RSB_M3, R_DIAG1 to R_DIAG2, R_VCC2 to R_VCC3, U2 to U3
Changed lines of the file:
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@@
 		(in_pos_files yes)
 		(dnp no)
-		(property "Reference" "C_BRB_FILT2"
+		(property "Reference" "C_BRB_FILT3"
 			(at 219.25 137.97 0)
 			(show_name no)
@@
 		(dnp no)
 		(fields_autoplaced yes)
-		(property "Reference" "#PWR053"
+		(property "Reference" "#PWR054"
 			(at 151.13 15.24 0)
 			(hide yes)
@@
 		(dnp no)
 		(fields_autoplaced yes)
-		(property "Reference" "#PWR029"
+		(property "Reference" "#PWR030"
 			(at 121.92 93.98 0)
 			(hide yes)
@@
 		(dnp no)
 		(fields_autoplaced yes)
-		(property "Reference" "#PWR051"
+		(property "Reference" "#PWR052"
 			(at 176.53 39.37 0)
 			(hide yes)
@@
 		(dnp no)
 		(fields_autoplaced yes)
-		(property "Reference" "#PWR039"
+		(property "Reference" "#PWR040"
 			(at 213.36 106.68 0)
 			(hide yes)
@@
 		(in_pos_files yes)
 		(dnp no)
-		(property "Reference" "U2"
+		(property "Reference" "U3"
 			(at 136.652 53.34 0)
 			(show_name no)
@@
 		(in_pos_files yes)
 		(dnp no)
-		(property "Reference" "C_5VOUT2"
+		(property "Reference" "C_5VOUT3"
 			(at 173.53 57.96 0)
 			(show_name no)
@@
 		(in_pos_files yes)
 		(dnp no)
-		(property "Reference" "C_VCC2"
+		(property "Reference" "C_VCC3"
 			(at 154.13 24.94 0)
 			(show_name no)
@@
 		(in_pos_files yes)
 		(dnp no)
-		(property "Reference" "RSA2"
+		(property "Reference" "RSA3"
 			(at 196.39 103.68 0)
 			(show_name no)
@@
 		(dnp no)
 		(fields_autoplaced yes)
-		(property "Reference" "#PWR045"
+		(property "Reference" "#PWR046"
 			(at 234.95 92.71 0)
 			(hide yes)
@@
 		(in_pos_files yes)
 		(dnp no)
-		(property "Reference" "R_VCC2"
+		(property "Reference" "R_VCC3"
 			(at 186.69 63.5 90)
 			(show_name no)
@@
 		(dnp no)
 		(fields_autoplaced yes)
-		(property "Reference" "#PWR063"
+		(property "Reference" "#PWR064"
 			(at 133.35 88.9 0)
 			(hide yes)
@@
 		(dnp no)
 		(fields_autoplaced yes)
-		(property "Reference" "#PWR023"
+		(property "Reference" "#PWR024"
 			(at 123.19 60.96 0)
 			(hide yes)
@@
 		(in_pos_files yes)
 		(dnp no)
-		(property "Reference" "C_BRA_FILT2"
+		(property "Reference" "C_BRA_FILT3"
 			(at 219.25 89.71 0)
 			(show_name no)
@@
 		(dnp no)
 		(fields_autoplaced yes)
-		(property "Reference" "#PWR057"
+		(property "Reference" "#PWR058"
 			(at 127 52.07 0)
 			(hide yes)
@@
 		(dnp no)
 		(fields_autoplaced yes)
-		(property "Reference" "#PWR019"
+		(property "Reference" "#PWR020"
 			(at 153.67 161.29 0)
 			(hide yes)
@@
 		(in_pos_files yes)
 		(dnp no)
-		(property "Reference" "RSB2"
+		(property "Reference" "RSB3"
 			(at 196.39 116.38 0)
 			(show_name no)
@@
 		(dnp no)
 		(fields_autoplaced yes)
-		(property "Reference" "#PWR061"
+		(property "Reference" "#PWR062"
 			(at 198.12 45.72 0)
 			(hide yes)
@@
 		(dnp no)
 		(fields_autoplaced yes)
-		(property "Reference" "#PWR017"
+		(property "Reference" "#PWR018"
 			(at 151.13 161.29 0)
 			(hide yes)
@@
 		(dnp no)
 		(fields_autoplaced yes)
-		(property "Reference" "#PWR021"
+		(property "Reference" "#PWR022"
 			(at 156.21 161.29 0)
 			(hide yes)
@@
 		(in_pos_files yes)
 		(dnp yes)
-		(property "Reference" "RSA_M2"
+		(property "Reference" "RSA_M3"
 			(at 196.39 93.52 0)
 			(show_name no)
@@
 		(in_pos_files yes)
 		(dnp no)
-		(property "Reference" "C_CP2"
+		(property "Reference" "C_CP3"
 			(at 179.53 130.35 0)
 			(show_name no)
@@
 		(in_pos_files yes)
 		(dnp no)
-		(property "Reference" "C_VCC_IO2"
+		(property "Reference" "C_VCC_IO3"
 			(at 130 37.64 0)
 			(show_name no)
@@
 		(in_pos_files yes)
 		(dnp no)
-		(property "Reference" "R_DIAG1"
+		(property "Reference" "R_DIAG2"
 			(at 213.82 64.31 0)
 			(show_name no)
@@
 		(dnp no)
 		(fields_autoplaced yes)
-		(property "Reference" "#PWR031"
+		(property "Reference" "#PWR032"
 			(at 121.92 96.52 0)
 			(hide yes)
@@
 		(in_pos_files yes)
 		(dnp no)
-		(property "Reference" "C_VSA2"
+		(property "Reference" "C_VSA3"
 			(at 227.79 28.75 0)
 			(show_name no)
@@
 		(in_pos_files yes)
 		(dnp yes)
-		(property "Reference" "RSB_M2"
+		(property "Reference" "RSB_M3"
 			(at 196.39 127.81 0)
 			(show_name no)
@@
 		(in_pos_files yes)
 		(dnp no)
-		(property "Reference" "C_VS_BULK2"
+		(property "Reference" "C_VS_BULK3"
 			(at 212.55 28.75 0)
 			(show_name no)
@@
 		(dnp no)
 		(fields_autoplaced yes)
-		(property "Reference" "#PWR013"
+		(property "Reference" "#PWR016"
 			(at 148.59 161.29 0)
 			(hide yes)
@@
 		(dnp no)
 		(fields_autoplaced yes)
-		(property "Reference" "#PWR055"
+		(property "Reference" "#PWR056"
 			(at 127 36.83 0)
 			(hide yes)
@@
 		(in_pos_files yes)
 		(dnp no)
-		(property "Reference" "C_VS2"
+		(property "Reference" "C_VS3"
 			(at 201.12 28.75 0)
 			(show_name no)
@@
 		(dnp no)
 		(fields_autoplaced yes)
-		(property "Reference" "#PWR041"
+		(property "Reference" "#PWR042"
 			(at 213.36 119.38 0)
 			(hide yes)
@@
 		(dnp no)
 		(fields_autoplaced yes)
-		(property "Reference" "#PWR059"
+		(property "Reference" "#PWR060"
 			(at 198.12 27.94 0)
 			(hide yes)
@@
 		(dnp no)
 		(fields_autoplaced yes)
-		(property "Reference" "#PWR049"
+		(property "Reference" "#PWR050"
 			(at 156.21 46.99 0)
 			(hide yes)
@@
 		(dnp no)
 		(fields_autoplaced yes)
-		(property "Reference" "#PWR047"
+		(property "Reference" "#PWR048"
 			(at 234.95 140.97 0)
 			(hide yes)
@@
 		(dnp no)
 		(fields_autoplaced yes)
-		(property "Reference" "#PWR043"
+		(property "Reference" "#PWR044"
 			(at 213.36 130.81 0)
 			(hide yes)
@@
 		(dnp no)
 		(fields_autoplaced yes)
-		(property "Reference" "#PWR027"
+		(property "Reference" "#PWR028"
 			(at 124.46 137.16 0)
 			(hide yes)
@@
 		(dnp no)
 		(fields_autoplaced yes)
-		(property "Reference" "#PWR037"
+		(property "Reference" "#PWR038"
 			(at 213.36 96.52 0)
 			(hide yes)
@@
 		(dnp no)
 		(fields_autoplaced yes)
-		(property "Reference" "#PWR033"
+		(property "Reference" "#PWR034"
 			(at 189.23 60.96 0)
 			(hide yes)
@@
 		(dnp no)
 		(fields_autoplaced yes)
-		(property "Reference" "#PWR035"
+		(property "Reference" "#PWR036"
 			(at 210.82 64.77 0)
 			(hide yes)
@@
 		(in_pos_files yes)
 		(dnp no)
-		(property "Reference" "C_VCP2"
+		(property "Reference" "C_VCP3"
 			(at 179.53 37.64 0)
 			(show_name no)
