File: hardware/ministepper/ministepper.kicad_sch (KiCad schematic)
At the start: 20 parts, among them J2 TC2030_NL, U1 STM32G0B1KBU6, U4 SIT3088EEUA

Commit message: Checkpoint
Parts:
- removed JP2: BOOT, Jumper:SolderJumper-2_P1.3mm_Open_Pad1.0x1.5mm, symbol Jumper:SolderJumper_2_Open
- renumbered C_MCU_BULK to C_MCU_BULK2, C_MCU_VDD to C_MCU_VDD2, C_NRST to C_NRST2, J_USB to J_USB2, SW_BOOT to SW_BOOT2
Connections:
- net +3.3V: now also C_MCU_BULK2.1, C_MCU_VDD2.1, SW_BOOT2.2, U1.4 (VDD/VDDA)
- net GND: now also C_MCU_BULK2.2, C_MCU_VDD2.2, J_USB2.A1 (GND), J_USB2.A12 (GND), J_USB2.B1 (GND), J_USB2.B12 (GND), J_USB2.SH (SHIELD), R_CC1.1, R_CC2.2, U1.33 (VSS), U1.5 (VSS/VSSA)
- net Stepper 1/MOT_A+: now also JMOT1.1 (Pin_1)
- net Stepper 1/MOT_A-: now also JMOT1.2 (Pin_2)
- net Stepper 1/MOT_B+: now also JMOT1.3 (Pin_3)
- net Stepper 1/MOT_B-: now also JMOT1.4 (Pin_4)
- net Stepper 2/MOT_A+: now also JMOT2.1 (Pin_1)
- net Stepper 2/MOT_A-: now also JMOT2.2 (Pin_2)
- net Stepper 2/MOT_B+: now also JMOT2.3 (Pin_3)
- net Stepper 2/MOT_B-: now also JMOT2.4 (Pin_4)
- net SWDIO: now reaches J2.2 (SWDIO)
- net SWDIO: now also U1.24 (PA13/SWDIO)
- net RST: now reaches J2.3 (~{RESET}), R5.2
- net RST: now also U1.6 (PF2/NRST)
- net SWCLK: now reaches J2.4 (SWCLK), R_BOOT0.1
- net SWCLK: now also SW_BOOT2.1, U1.25 (PA14/SWCLK/BOOT0)
- net RX: now reaches U1.10 (PA3)
- net CS1: now reaches U1.11 (PA4)
- net SCK: now reaches U1.12 (PA5)
- net MISO: now reaches U1.13 (PA6)
- net MOSI: now reaches U1.14 (PA7)
- net LIM1: now reaches U1.15 (PB0)
- net DIAG1: now reaches U1.16 (PB1)
- net DRV_ENNN: now reaches U1.17 (PB2)
- net STEP1: now reaches U1.18 (PA8)
- net CS2: now reaches U1.19 (PA9)
- net DIR2: now reaches U1.20 (PC6)
- net USBDM: now reaches U1.22 (PA11)
- net USBDM: now also J_USB2.A7 (D-), J_USB2.B7 (D-)
- net USBDP: now reaches U1.23 (PA12)
- net USBDP: now also J_USB2.A6 (D+), J_USB2.B6 (D+)
- net DIR1: now reaches U1.26 (PA15)
- net LIM2: now reaches U1.27 (PB3)
- net DIAG2: now reaches U1.28 (PB4)
- net LED: now reaches U1.29 (PB5)
- net SCL: now reaches U1.30 (PB6)
- net SDA: now reaches U1.31 (PB7)
- net STEP2: now reaches U1.7 (PA0)
- net DE: now reaches U1.8 (PA1)
- net TX: now reaches U1.9 (PA2)
- net at R_CC2.1: now also J_USB2.A5 (CC1)
- net at J_USB2.B5 (CC2): now also R_CC1.2
Other:
- moved on the sheet: C_MCU_VDD2, C_NRST2, J2, JBUS1, JBUS2, JMOT1, JMOT2, J_USB2, R5, R_BOOT0, R_CC1, R_CC2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
