File: hardware/ministepper/ministepper.kicad_pcb (KiCad board)
At the start: 4 copper layers, 52 parts, among them U1 STM32G071G8U6, U2 TMC2130-LA, U3 TMC2130-LA, U4 SIT3088EEUA, U9 TPS54061DRBT

Commit message: Checkpoint
Parts:
- added C_MCU_BULK2: 4.7uF, Capacitor_SMD:C_0603_1608Metric, F.Cu at (128.8, 127.1)
- added C_MCU_VDD2: 100nF, Capacitor_SMD:C_0402_1005Metric, F.Cu at (132.5, 123.3)
- added C_NRST2: 100nF, Capacitor_SMD:C_0402_1005Metric, F.Cu at (132.5, 125.2)
- added J2: TC2030_NL, Connector:Tag-Connect_TC2030-IDC-NL_2x03_P1.27mm_Vertical, F.Cu at (122.7, 124.8)
- added J_USB2: USB-TYPE-C-019, Connector_USB:USB_C_Receptacle_GCT_USB4105-xx-A_16P_TopMnt_Horizontal, F.Cu at (124.5, 117.6)
- added R5: 10k, Resistor_SMD:R_0402_1005Metric, F.Cu at (131.8, 113.3)
- added R_BOOT0: 10k, Resistor_SMD:R_0402_1005Metric, F.Cu at (131.8, 115.3)
- added R_CC1: 5.1k, Resistor_SMD:R_0402_1005Metric, F.Cu at (131.8, 117.3)
- added R_CC2: 5.1k, Resistor_SMD:R_0402_1005Metric, F.Cu at (131.8, 119.3)
- added SW_BOOT2: TS-1187A, tsumikoro:SW_Push_1P1T_XKB_TS-1187A, F.Cu at (149.4, 125.6)
- D1, D2: value SS34 -> SS54
- U1: value STM32G071G8U6 -> STM32G0B1KBU6; footprint tsumikoro:UFQFPN-28 -> tsumikoro:UFQFPN-32
- moved U3 114.0 mm to (78.9, 109.4)
- moved C_VCC_IO3 113.2 mm to (74.3, 111.2), turned to -90 degrees
- moved R_VCC3 112.1 mm to (83.5, 109.1), turned to 90 degrees
- moved C_BRB_FILT3 111.4 mm to (75.9, 116.7), turned to -90 degrees
- moved R_DIAG2 110.8 mm to (84.3, 110.5), turned to 180 degrees
- moved C_5VOUT2 108.9 mm to (85.2, 83.3)
- moved C_BRA_FILT2 108.9 mm to (81.2, 75.3)
- moved C_BRB_FILT2 108.9 mm to (75.7, 90.7)
- moved C_CP2 108.9 mm to (83.2, 81.2)
- moved C_VCC2 108.9 mm to (85.2, 81.7)
- moved C_VS2 108.9 mm to (81.0, 89.3)
- moved RSA2 108.9 mm to (78.8, 75.3)
- moved RSB2 108.9 mm to (78.2, 90.7)
- moved R_VCC2 108.9 mm to (83.2, 83.1)
- moved C_VCC_IO2 108.9 mm to (74.0, 85.2)
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Connections:
- JMOT1 pad 1: unconnected-(JMOT1-Pin_1-Pad1) -> /Stepper 1/MOT_A+
- JMOT1 pad 2: unconnected-(JMOT1-Pin_2-Pad2) -> /Stepper 1/MOT_A-
- JMOT1 pad 3: unconnected-(JMOT1-Pin_3-Pad3) -> /Stepper 1/MOT_B+
- JMOT1 pad 4: unconnected-(JMOT1-Pin_4-Pad4) -> /Stepper 1/MOT_B-
- JMOT2 pad 1: unconnected-(JMOT2-Pin_1-Pad1) -> /Stepper 2/MOT_A+
- JMOT2 pad 2: unconnected-(JMOT2-Pin_2-Pad2) -> /Stepper 2/MOT_A-
- JMOT2 pad 3: unconnected-(JMOT2-Pin_3-Pad3) -> /Stepper 2/MOT_B+
- JMOT2 pad 4: unconnected-(JMOT2-Pin_4-Pad4) -> /Stepper 2/MOT_B-
- R_DIAG1 pad 2: /Stepper 1/DIAG1 -> /DIAG1
- R_DIAG2 pad 2: /Stepper 2/DIAG1 -> /DIAG2
- U1 pad 10: unconnected-(U1-PA6-Pad10) -> /RX
- U1 pad 11: unconnected-(U1-PA7-Pad11) -> /CS1
- U1 pad 12: unconnected-(U1-PA8-Pad12) -> /SCK
- U1 pad 13: unconnected-(U1-PA11-Pad13) -> /MISO
- U1 pad 14: unconnected-(U1-PA12-Pad14) -> /MOSI
- U1 pad 15: unconnected-(U1-PA13/SWDIO-Pad15) -> /LIM1
- U1 pad 16: unconnected-(U1-PA14/SWCLK-Pad16) -> /DIAG1
- U1 pad 17: unconnected-(U1-PA15-Pad17) -> /DRV_ENNN
- U1 pad 18: unconnected-(U1-PB0-Pad18) -> /STEP1
- U1 pad 19: unconnected-(U1-PB1-Pad19) -> /CS2
- U1 pad 20: unconnected-(U1-PB2-Pad20) -> /DIR2
- U1 pad 22: unconnected-(U1-PB4-Pad22) -> /USBDM
- U1 pad 23: unconnected-(U1-PB5-Pad23) -> /USBDP
- U1 pad 24: unconnected-(U1-PB6-Pad24) -> /SWDIO
- U1 pad 25: unconnected-(U1-PB7-Pad25) -> /SWCLK
- U1 pad 26: unconnected-(U1-PB8-Pad26) -> /DIR1
- U1 pad 27: unconnected-(U1-VSS-Pad27) -> /LIM2
- U1 pad 28: unconnected-(U1-VDD_2-Pad28) -> /DIAG2
- U1 pad 29: unconnected-(U1-EP-Pad29) -> /LED
- U1 pad 4: unconnected-(U1-PA0-Pad4) -> +3.3V
- U1 pad 5: unconnected-(U1-PA1-Pad5) -> GND
- U1 pad 6: unconnected-(U1-PA2-Pad6) -> /RST
- U1 pad 7: unconnected-(U1-PA3-Pad7) -> /STEP2
- U1 pad 8: unconnected-(U1-PA4-Pad8) -> /DE
- U1 pad 9: unconnected-(U1-PA5-Pad9) -> /TX
- U2 pad 2: /Stepper 1/CS -> /CS1
- U2 pad 21: /Stepper 1/DIAG1 -> /DIAG1
- U2 pad 22: /Stepper 1/DRV_ENN -> /DRV_ENN
- U2 pad 3: /Stepper 1/SCK -> /SCK
- U2 pad 4: /Stepper 1/MOSI -> /MOSI
- U2 pad 5: /Stepper 1/MISO -> /MISO
- U2 pad 6: /Stepper 1/STEP -> /STEP1
- U2 pad 7: /Stepper 1/DIR -> /DIR1
- U3 pad 2: /Stepper 2/CS -> /CS2
- U3 pad 21: /Stepper 2/DIAG1 -> /DIAG2
- U3 pad 22: /Stepper 2/DRV_ENN -> /DRV_ENN
- U3 pad 3: /Stepper 2/SCK -> /SCK
- U3 pad 4: /Stepper 2/MOSI -> /MOSI
- U3 pad 5: /Stepper 2/MISO -> /MISO
- U3 pad 6: /Stepper 2/STEP -> /STEP2
- U3 pad 7: /Stepper 2/DIR -> /DIR2
Routing:
- net GND: track 7.25 -> 57.3 mm, vias 1 -> 74
- net /MISO: track 0.00 -> 35.0 mm, vias 0 -> 2
- net /SCK: track 0.00 -> 34.3 mm, vias 0 -> 2
- net /MOSI: track 0.00 -> 33.0 mm, vias 0 -> 2
- net /CS1: track 0.00 -> 26.2 mm, vias 0 -> 2
- net /DIR1: track 0.00 -> 24.4 mm, vias 0 -> 1
- net VPP: track 5.48 -> 21.9 mm
- net /Stepper 1/MOT_A-: track 0.00 -> 15.6 mm, vias 0 -> 1
- net /Stepper 2/MOT_A-: track 0.00 -> 15.5 mm, vias 0 -> 1
- net /Stepper 1/MOT_A+: track 0.00 -> 13.9 mm
- net /Stepper 2/MOT_B-: track 0.00 -> 13.4 mm, vias 0 -> 1
- net /Stepper 1/MOT_B-: track 0.00 -> 13.2 mm, vias 0 -> 1
- net /Stepper 2/MOT_B+: track 0.00 -> 12.8 mm
- net /Stepper 1/MOT_B+: track 0.00 -> 12.7 mm
- net /Stepper 2/MOT_A+: track 0.00 -> 12.3 mm
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- added copper zone on F.Cu, net GND
